File: Hardware/shori/shori.kicad_sch (KiCad schematic)
At the start: 100 parts, among them J1 430450200, J2 SWD_Header, J3 UART_Header, J4 530480310, J5 AudioJack3, J6 530480210, U1 CS4272, U2 STM32H750VBTx, U3 NE5532, U4 NE5532, U5 TPS73733DCQR, U6 OPA134, Y1 16MHz

Commit message: Layout complete!!!!!!
Next is setting up the board border and rounded corners, change the molex power connector to JST one. and start routing!!
Parts:
- J2: footprint Connector_PinHeader_2.54mm:PinHeader_1x05_P2.54mm_Vertical -> Connector_PinHeader_2.54mm:PinHeader_1x04_P2.54mm_Vertical
- J3: footprint Connector_JST:JST_XH_S4B-XH-A-1_1x04_P2.50mm_Horizontal -> MyFootprints:CONN04_530480410_MOL
Connections:
- net +5V: now also J1.2; no longer J1.1
- net AUDIO_OUT: now also J6.2; no longer J6.1
- net GND: now also J1.1, J6.1; no longer J1.2, J6.2
- net UART_RX: now also R14.1; no longer R10.2
- net UART_RX_RES: now also R14.2, U2.37 (PE7); no longer R10.1, U2.23 (PA1)
- net UART_TX: now also R10.1; no longer R14.2
- net UART_TX_RES: now also R10.2, U2.38 (PE8); no longer R14.1, U2.22 (PA0)
Other:
- moved on the sheet: C13, C14, C21, C33, Y1
