File: Hardware/shori/shori.kicad_sch (KiCad schematic)
At the start: 134 parts, among them J1 430450200, J2 Conn_01x05_Pin, J3 UART_Header, J4 530480310, J5 Conn_01x03, J6 530480310, J7 GROUND PROBE, SW1 SW_SPDT, U1 CS4272, U2 STM32H750VBTx, U3 NE5532, U4 NE5532, U5 TPS73733DCQR, U6 W25Q128JVS, U7 TLV9001IDCK, Y1 12.288MHz

Commit message: added stiching vias on gen and changed SWD header on shori to header pins
Parts:
- removed R40: 10Ω, Resistor_SMD:R_0402_1005Metric_Pad0.72x0.64mm_HandSolder, symbol Device:R
- C15: value 47uF -> 100uF
- J2: footprint Connector_Molex:Molex_PicoBlade_53048-0510_1x05_P1.25mm_Horizontal -> Connector_PinHeader_2.54mm:PinHeader_1x05_P2.54mm_Vertical
- J3: footprint MyFootprints:CONN04_530480410_MOL -> MyFootprints:MOLEX_530480310
Connections:
- net +5VA is gone; now on net +5V: C15.1, C24.1, C49.1, C50.2, R4.1, TP4.1, U1.20 (VA), U3.8 (V+), U4.8 (V+), U7.5 (V+)
- net +3.3V: now also U2.6 (VBAT)
- no-connect marks 75 -> 74
Changed lines of the file:
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@@
 	)
 	(no_connect
-		(at 151.13 243.84)
-	)
-	(no_connect
 		(at 449.58 236.22)
 	)
@@
 	(wire
 		(pts
-			(xy 566.42 314.96) (xy 566.42 317.5)
-		)
-		(stroke
-			(width 0)
-			(type default)
-		)
-	)
-	(wire
-		(pts
 			(xy 449.58 85.09) (xy 449.58 91.44)
 		)
@@
 	(wire
 		(pts
-			(xy 566.42 325.12) (xy 566.42 327.66)
-		)
-		(stroke
-			(width 0)
-			(type default)
-		)
-	)
-	(wire
-		(pts
 			(xy 57.15 204.47) (xy 57.15 215.9)
 		)
@@
 	(wire
 		(pts
+			(xy 148.59 243.84) (xy 151.13 243.84)
+		)
+		(stroke
+			(width 0)
+			(type default)
+		)
+	)
+	(wire
+		(pts
 			(xy 223.52 264.16) (xy 223.52 287.02)
 		)
@@
 	(wire
 		(pts
+			(xy 566.42 314.96) (xy 566.42 327.66)
+		)
+		(stroke
+			(width 0)
+			(type default)
+		)
+	)
+	(wire
+		(pts
 			(xy 566.42 327.66) (xy 560.07 327.66)
 		)
@@
 			)
 		)
-		(property "Footprint" "MyFootprints:CONN04_530480410_MOL"
+		(property "Footprint" "MyFootprints:MOLEX_530480310"
 			(at 247.65 356.87 0)
 			(hide yes)
@@
 			)
 		)
-		(property "Value" "47uF"
+		(property "Value" "100uF"
 			(at 539.6383 334.3009 0)
 			(show_name no)
@@
 	(symbol
 		(lib_id "Device:R")
-		(at 566.42 321.31 0)
-		(mirror x)
-		(unit 1)
-		(body_style 1)
-		(exclude_from_sim no)
-		(in_bom yes)
-		(on_board yes)
-		(in_pos_files yes)
-		(dnp no)
-		(property "Reference" "R40"
-			(at 563.88 320.294 90)
-			(show_name no)
-			(do_not_autoplace no)
-			(effects
-				(font
-					(size 1.27 1.27)
-				)
-				(justify left)
-			)
-		)
-		(property "Value" "10Ω"
-			(at 568.706 320.04 90)
-			(show_name no)
-			(do_not_autoplace no)
-			(effects
-				(font
-					(size 1.27 1.27)
-				)
-				(justify left)
-			)
-		)
-		(property "Footprint" "Resistor_SMD:R_0402_1005Metric_Pad0.72x0.64mm_HandSolder"
-			(at 564.642 321.31 90)
-			(hide yes)
-			(show_name no)
-			(do_not_autoplace no)
-			(effects
-				(font
-					(size 1.27 1.27)
-				)
-			)
-		)
-		(property "Datasheet" ""
-			(at 566.42 321.31 0)
-			(hide yes)
-			(show_name no)
-			(do_not_autoplace no)
-			(effects
-				(font
-					(size 1.27 1.27)
-				)
-			)
-		)
-		(property "Description" "Resistor"
-			(at 566.42 321.31 0)
-			(hide yes)
-			(show_name no)
-			(do_not_autoplace no)
-			(effects
-				(font
-					(size 1.27 1.27)
-				)
-			)
-		)
-		(property "KLC_S3.3" ""
-			(at 566.42 321.31 90)
-			(hide yes)
-			(show_name no)
-			(do_not_autoplace no)
-			(effects
-				(font
-					(size 1.27 1.27)
-				)
-			)
-		)
-		(property "KLC_S4.1" ""
-			(at 566.42 321.31 90)
-			(hide yes)
-			(show_name no)
-			(do_not_autoplace no)
-			(effects
-				(font
-					(size 1.27 1.27)
-				)
-			)
-		)
-		(pin "1"
-		)
-		(pin "2"
-		)
-		(instances
-			(project "shori"
-				(path "/bed06ac2-3d53-4627-b912-3f6150ebe2ee"
-					(reference "R40")
-					(unit 1)
-				)
-			)
-		)
-	)
-	(symbol
-		(lib_id "Device:R")
 		(at 367.03 274.32 180)
 		(unit 1)
@@
 			)
 		)
-		(property "Footprint" "Connector_Molex:Molex_PicoBlade_53048-0510_1x05_P1.25mm_Horizontal"
+		(property "Footprint" "Connector_PinHeader_2.54mm:PinHeader_1x05_P2.54mm_Vertical"
 			(at 54.61 289.56 0)
 			(hide yes)
