File: Hardware/shoyu/shoyu.kicad_sch (KiCad schematic)
At the start: 0 parts

Commit message: Shoyu: schems started, power input and output conns added
Parts:
- added J1: 5/9V Connector, symbol Connector_Generic:Conn_01x04
- added J2: 24V Connector, symbol Connector_Generic:Conn_01x03
- added J3: SHORI OUT, symbol Connector_Generic:Conn_01x02
- added J4: GAMEN_OUT, symbol Connector_Generic:Conn_01x02
- added J5: MAE OUT, symbol Connector_Generic:Conn_01x02
Connections:
- new net +24V: J2.2 (Pin_2)
- new net +5V: J1.2 (Pin_2), J3.2 (Pin_2), J4.2 (Pin_2)
- new net +9V: J1.4 (Pin_4), J5.1 (Pin_1)
- new net GND: J1.1 (Pin_1), J1.3 (Pin_3), J2.1 (Pin_1), J2.3 (Pin_3), J3.1 (Pin_1), J4.1 (Pin_1), J5.2 (Pin_2)

Commit message: Shoyu: Schems finished Footpritns added
Parts:
- added C1, C2, C32, C33, C34, C36: 100uF, Capacitor_THT:CP_Radial_D8.0mm_P3.50mm, symbol Device:C_Polarized
- added C10, C19, C20, C27, C28, C29, C30, C39, C8, C9: 1uF, Capacitor_SMD:C_0603_1608Metric_Pad1.08x0.95mm_HandSolder, symbol Device:C
- added C11, C23, C24, C25: 33nF, Capacitor_SMD:C_0402_1005Metric_Pad0.74x0.62mm_HandSolder, symbol Device:C
- added C12: 47nF, Capacitor_SMD:C_0402_1005Metric_Pad0.74x0.62mm_HandSolder, symbol Device:C
- added C13, C14, C35, C37, C4, C5: 100nF, Capacitor_SMD:C_0402_1005Metric_Pad0.74x0.62mm_HandSolder, symbol Device:C
- added C15, C16, C17, C18: 470nF, Capacitor_SMD:C_0402_1005Metric_Pad0.74x0.62mm_HandSolder, symbol Device:C
- added C21, C22: 10nF, Capacitor_SMD:C_0402_1005Metric_Pad0.74x0.62mm_HandSolder, symbol Device:C
- added C26, C3, C31: 470uF, Capacitor_THT:CP_Radial_D10.0mm_P5.00mm, symbol Device:C_Polarized
- added C38: 1000uF, Capacitor_THT:CP_Radial_D12.5mm_P5.00mm, symbol Device:C_Polarized
- added C6, C7: 10uF, Capacitor_SMD:C_0805_2012Metric_Pad1.18x1.45mm_HandSolder, symbol Device:C
- added J6: AUDIO IN, Connector_JST:JST_PH_S2B-PH-K_1x02_P2.00mm_Horizontal, symbol Connector_Generic:Conn_01x02
- added L1, L2: 10uH, My Feet pics:IND_SRP1038A_BRN-M, symbol Device:L
- added LS1: Speaker, symbol Device:Speaker
- added R1, R5, R7, R8: 3.3Ω, Resistor_SMD:R_0402_1005Metric_Pad0.72x0.64mm_HandSolder, symbol Device:R
- added R3: 22K, Resistor_SMD:R_0402_1005Metric_Pad0.72x0.64mm_HandSolder, symbol Device:R
- added R4: 33K, Resistor_SMD:R_0402_1005Metric_Pad0.72x0.64mm_HandSolder, symbol Device:R
- added R6: 10K, Resistor_SMD:R_0402_1005Metric_Pad0.72x0.64mm_HandSolder, symbol Device:R
- added TP1, TP2: TestPoint, symbol Connector:TestPoint
- added U1: TPA3255DDVR, Package_SO:HTSSOP-44_6.1x14mm_P0.635mm_TopEP4.14x7.01mm, symbol My Symbols:TPA3255DDVR
- added U10, U9: (no value), Package_TO_SOT_SMD:SOT-23-3, symbol MyCrystal:ESDS452DBZRQ1
- added U2: TSR 1-24120, My Footprints:TSR1-SINGLE_TRP, symbol My Symbols:TSR_1-24120
- J1: footprint (none) -> Connector_JST:JST_XH_S4B-XH-A_1x04_P2.50mm_Horizontal
- J2: footprint (none) -> Connector_JST:JST_XH_S3B-XH-A_1x03_P2.50mm_Horizontal
- J3, J4, J5: footprint (none) -> Connector_JST:JST_XH_S2B-XH-A_1x02_P2.50mm_Horizontal
Connections:
- net +24V: now also C1.1, C26.1, C27.2, C28.1, C29.2, C30.1, C31.1, C38.1, C39.1, U1.29 (PVDD_CD_29), U1.30 (PVDD_CD_30), U1.31 (PVDD_CD_31), U1.36 (PVDD_AB_36), U1.37 (PVDD_AB_37), U1.38 (PVDD_AB_38), U2.1 (+VIN)
- net +5V: now also C14.1, C33.1, C34.1, C35.1
- net +9V: now also C36.1, C37.1
- net GND: now also C1.2, C10.2, C12.2, C13.1, C14.2, C15.1, C16.2, C17.2, C18.1, C19.1, C2.2, C20.2, C26.2, C27.1, C28.2, C29.1, C3.2, C30.2, C31.2, C32.2, C33.2, C34.2, C35.2, C36.2, C37.2, C38.2, C39.2, C4.2, C5.2, C8.2, C9.2, R3.1, R4.1, R7.2, R8.1, U1.12 (GND_12), U1.13 (GND_13), U1.16 (INPUT_C), U1.17 (INPUT_D), U1.25 (GND_25), U1.26 (GND_26), U1.3 (M1), U1.33 (GND_33), U1.34 (GND_34), U1.41 (GND_41), U1.42 (GND_42), U10.3 (GND), U2.2 (GND), U9.3 (GND)
- new net: C6.1, J6.2 (Pin_2), U10.1 (IO1)
- new net: C6.2, U1.5 (INPUT_A)
- new net: C15.2, C18.2, C19.2, C21.2, L2.2, LS1.1
- new net: C23.1, C24.2, L1.1, U1.27 (OUT_D_27), U1.28 (OUT_D_28), U1.35 (OUT_B)
- new net: C16.1, C17.1, C20.1, C22.1, L1.2, LS1.2
- new net: TP1.1, U1.19 (~{FAULT})
- new net: C7.1, J6.1 (Pin_1), U9.2 (IO2)
- new net: C11.2, C25.1, L2.1, U1.32 (OUT_C), U1.39 (OUT_A_39), U1.40 (OUT_A_40)
- new net: C22.2, R8.2
- new net: C32.1, R6.1, U1.18 (~{RESET})
- new net: C21.1, R7.1
- new net: C7.2, U1.6 (INPUT_B)
- new net: C5.1, R1.2, U1.1 (GVDD_AB)
- new net: R3.2, U1.7 (OC_ADJ)
- new net: C8.1, U1.14 (AVDD)
- new net: C13.2, R5.1, U1.22 (GVDD_CD)
- new net: C9.1, U1.11 (DVDD)
- new net: C12.1, U1.15 (C_START)
- new net: TP2.1, U1.21 (~{CLIP_OTW})
- new net: R4.2, U1.8 (FREQ_ADJ)
- new net +12V: C2.1, C3.1, C4.1, R1.1, R5.2, R6.2, U1.2 (VDD), U2.3 (+VOUT)
- new net BST_A: C11.1, U1.44 (BST_A)
- new net BST_B: C23.2, U1.43 (BST_B)
- new net BST_C: C25.2, U1.24 (BST_C)
- new net BST_D: C24.1, U1.23 (BST_D)
- new net CHIP_M2: C10.1, U1.20 (VBG), U1.4 (M2)
- no-connect marks 0 -> 6
Other:
- note added: "24 -> 12V CONVERTOR"
- note added: "CONNECTOR DECOUPLING"
- note added: "POWER AMP + AUDIO IN + SPEAKER"
- note added: "POWER INPUT AND OUTPUT"
- note added: "SHOYU REV ONE"
- note added: "WAVE FORGE"
- moved on the sheet: J1, J2, J3, J4, J5

Commit message: Shoyu: Layout complete
Parts:
- added H1, H2, H3, H4: MountingHole, MountingHole:MountingHole_2mm, symbol Mechanical:MountingHole
- C10, C8, C9: footprint Capacitor_SMD:C_0603_1608Metric_Pad1.08x0.95mm_HandSolder -> Capacitor_SMD:C_0603_1608Metric
- C27, C28, C29, C30: value 1uF -> 2.2uF; footprint Capacitor_SMD:C_0603_1608Metric_Pad1.08x0.95mm_HandSolder -> Capacitor_SMD:C_0603_1608Metric
- LS1: footprint (none) -> TerminalBlock_CUI:TerminalBlock_CUI_TB007-508-02_1x02_P5.08mm_Horizontal
- U2: footprint My Footprints:TSR1-SINGLE_TRP -> My Feet pics:TSR1-SINGLE_TRP
Connections:
- net +5V: now also J1.4 (Pin_4); no longer J1.2 (Pin_2)
- net +9V: now also J1.2 (Pin_2); no longer J1.4 (Pin_4)
- net at C6.1, U10.1 (IO1): now also J6.1 (Pin_1); no longer J6.2 (Pin_2)
- net at C7.1, U9.2 (IO2): now also J6.2 (Pin_2); no longer J6.1 (Pin_1)
Other:
- moved on the sheet: J6

Commit message: Shoyu: rev 1 routing complete
Connections:
- net AUDIO_IN+: now reaches C6.2, U1.5 (INPUT_A)
- net INDUCTOR_IN_L1: now reaches C23.1, C24.2, L1.1, U1.27 (OUT_D_27), U1.28 (OUT_D_28), U1.35 (OUT_B)
- net INDUCTOR_IN_L2: now reaches C11.2, C25.1, L2.1, U1.32 (OUT_C), U1.39 (OUT_A_39), U1.40 (OUT_A_40)
- net AUDIO_IN-: now reaches C7.2, U1.6 (INPUT_B)
Changed lines of the file:
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@@
+		)
+	)
+	(label "AUDIO_IN+"
+		(at 125.73 140.97 0)
+		(effects
+			(font
+				(size 1.27 1.27)
+			)
+			(justify left bottom)
 		)
 	)
@@
 		)
 	)
+	(label "AUDIO_IN-"
+		(at 125.73 149.86 0)
+		(effects
+			(font
+				(size 1.27 1.27)
+			)
+			(justify left bottom)
+		)
+	)
+	(label "INDUCTOR_IN_L2"
+		(at 231.14 151.13 0)
+		(effects
+			(font
+				(size 1.27 1.27)
+			)
+			(justify left bottom)
+		)
+	)
+	(label "INDUCTOR_IN_L1"
+		(at 231.14 158.75 0)
+		(effects
+			(font
+				(size 1.27 1.27)
+			)
+			(justify left bottom)
+		)
+	)

Commit message: Shoyu: New Film caps for output filter
Parts:
- C15, C16, C17, C18: footprint Capacitor_SMD:C_0402_1005Metric_Pad0.74x0.62mm_HandSolder -> Capacitor_THT:C_Rect_L7.2mm_W3.5mm_P5.00mm
Changed lines of the file:
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@@
 			)
 		)
-		(property "Footprint" "Capacitor_SMD:C_0402_1005Metric_Pad0.74x0.62mm_HandSolder"
+		(property "Footprint" "Capacitor_THT:C_Rect_L7.2mm_W3.5mm_P5.00mm"
 			(at 256.8448 138.43 0)
 			(hide yes)
@@
 			)
 		)
-		(property "Footprint" "Capacitor_SMD:C_0402_1005Metric_Pad0.74x0.62mm_HandSolder"
+		(property "Footprint" "Capacitor_THT:C_Rect_L7.2mm_W3.5mm_P5.00mm"
 			(at 274.6248 138.43 0)
 			(hide yes)
@@
 			)
 		)
-		(property "Footprint" "Capacitor_SMD:C_0402_1005Metric_Pad0.74x0.62mm_HandSolder"
+		(property "Footprint" "Capacitor_THT:C_Rect_L7.2mm_W3.5mm_P5.00mm"
 			(at 274.6248 153.67 0)
 			(hide yes)
@@
 			)
 		)
-		(property "Footprint" "Capacitor_SMD:C_0402_1005Metric_Pad0.74x0.62mm_HandSolder"
+		(property "Footprint" "Capacitor_THT:C_Rect_L7.2mm_W3.5mm_P5.00mm"
 			(at 256.8448 153.67 0)
 			(hide yes)
