File: Hardware/shori rev 4/shori.kicad_pcb (KiCad board)
At the start: 4 copper layers, 101.5 x 44.8 mm, 135 parts, among them J1 430450200, J2 Conn_01x05_Pin, J3 UART_Header, J4 530480310, J5 Conn_01x03, J6 530480210, J7 GROUND PROBE, SW1 SW_SPDT, U1 CS4272, U2 STM32H750VBTx, U3 NE5532, U4 NE5532, U5 TPS73733DCQR, U6 W25Q128JVS, U7 TLV9001IDCK, Y1 12.288MHz

Commit message: Shorr rev 4 completed and gamen started
Gamen is going to actually make me kill my self
Parts:
- removed J6: 530480210, My footprints:CONN02_530480210_MOL
- removed J7: GROUND PROBE, Connector_PinSocket_2.00mm:PinSocket_1x02_P2.00mm_Vertical
- added AUDIO OUT: 530480310, MyFootprints:MOLEX_530480310, F.Cu at (181.6, 95.9)
- added C52: 100pF, Capacitor_SMD:C_0402_1005Metric_Pad0.74x0.62mm_HandSolder, F.Cu at (175.7, 112.7)
- added C53: 10uF, Capacitor_SMD:C_0805_2012Metric, F.Cu at (174.0, 105.6)
- added GND: TestPoint_Bridge_Pitch2.54mm_Drill1.0mm, TestPoint:TestPoint_Bridge_Pitch2.54mm_Drill1.0mm, F.Cu at (103.8, 123.8)
- added R46: 10K, Resistor_SMD:R_0402_1005Metric_Pad0.72x0.64mm_HandSolder, F.Cu at (176.8, 112.8)
- AUDIO IN: renamed from J4
- AUX IN: renamed from J5
- C17, C29, C3, C30, C4, C40, C41, C47, C50, C51: footprint Capacitor_SMD:C_0603_1608Metric_Pad1.08x0.95mm_HandSolder -> Capacitor_SMD:C_0805_2012Metric
- C23, C43, C46: footprint Capacitor_SMD:C_0805_2012Metric -> Capacitor_SMD:C_1206_3216Metric
- moved C25 11.0 mm to (185.5, 111.4)
- moved C51 10.2 mm to (187.1, 110.9), turned to -90 degrees
- moved C29 8.89 mm to (176.1, 105.5), turned to 90 degrees
- moved C50 7.41 mm to (176.5, 116.1), turned to 180 degrees
- moved C24 6.55 mm to (177.8, 108.7), turned to 90 degrees
- moved R4 5.52 mm to (178.9, 108.7)
- moved C3 5.45 mm to (147.5, 122.5), turned to 0 degrees
- moved R5 3.86 mm to (181.2, 108.2)
- moved R9 2.74 mm to (187.0, 114.4), turned to -90 degrees
- moved R7 2.36 mm to (189.2, 114.9)
- moved C28 2.18 mm to (185.8, 114.3), turned to -90 degrees
- moved C27 2.15 mm to (191.0, 115.5)
- moved U4 1.73 mm to (181.2, 112.8)
- moved C42 1.64 mm to (162.8, 110.1), turned to 90 degrees
- moved U10 1.62 mm to (176.7, 127.9)
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- renumbered TP2 to 3V3, TP3 to 3V3A, TP1 to 5V, TP4 to 5VA, J2 to DEBUG, SW1 to P, J1 to POWER, J3 to UART
Connections:
- C28 pad 2: /SUMMED_OUT -> /SUMMED_OUT+
- C29 pad 1: /SUMMED_OUT -> /SUMMED_OUT+
- C29 pad 2: /AUDIO_OUT -> /AUDIO_OUT+
- R9 pad 2: /SUMMED_OUT -> /SUMMED_OUT+
- U10 pad 1: unconnected-(U10-IO1-Pad1) -> /SHUNT_RES_AINM
- U10 pad 2: /SHUNT_RES_AINM -> unconnected-(U10-IO2-Pad2)
- U15 pad 1: unconnected-(U15-IO1-Pad1) -> +5V
- U4 pad 1: /SUMMED_OUT -> /SUMMED_OUT+
- U4 pad 6: /UNUSED_INVERTOR -> /SUMMED_OUT+
- U4 pad 7: /UNUSED_INVERTOR -> /SUMMED_OUT-
- U9 pad 1: unconnected-(U9-IO1-Pad1) -> /SHUNT_RES_AINP
- U9 pad 2: /SHUNT_RES_AINP -> unconnected-(U9-IO2-Pad2)
Routing:
- net /SUMMED_OUT+: track 0.00 -> 18.4 mm, vias 0 -> 2
- net /AUDIO_OUT: track 12.4 -> 0.00 mm
- net /AUDIO_OUT-: track 0.00 -> 11.7 mm
- net /AUDIO_OUT+: track 0.00 -> 11.7 mm
- net /SUMMED_OUT: track 10.9 -> 0.00 mm, vias 2 -> 0
- net /SUMMED_OUT-: track 0.00 -> 10.5 mm
- net +5VA: track 67.7 -> 73.8 mm, vias 3 -> 4
- net +5V: track 25.0 -> 29.7 mm
- net GND: track 99.3 -> 96.1 mm, vias 157 -> 159
- net Net-(U3B-+): track 11.7 -> 14.1 mm
- net /JACKR: track 7.12 -> 4.92 mm
- net /AUDIO_IN+: track 6.36 -> 8.31 mm
- net /AUX_MIX: track 14.2 -> 12.5 mm
- net /UNUSED_INVERTOR: track 1.27 -> 0.00 mm
- net /VCOM: track 27.6 -> 26.5 mm
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